File: pcb/NumBLE.kicad_pcb (KiCad board)
At the start: 2 copper layers, 75.2 x 128.3 mm, 77 parts, among them J1 HRO_TYPE-C-31-M-12, J2 Conn_ARM_JTAG_SWD_10, J3 JST_S2B-PH-SM4-TB, Q1 AO3407, SW1 JS202011JCQN, SW2 KSC721J, SW3 RotaryEncoder_Switch, U1 USBLC6-2SC6, U2 MAX17263xxTE, U3 MCP73831-2-OT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

Commit message: Fix resistor numbering
Parts:
- U2: footprint Package_DFN_QFN:TDFN-14-1EP_3x3mm_P0.4mm_EP1.78x2.35mm -> Package_DFN_QFN:DFN-14-1EP_3x3mm_P0.4mm_EP1.78x2.35mm
- renumbered R7 to R6, R8 to R7
