File: pcb/NumBLE.kicad_sch (KiCad schematic)
At the start: 77 parts, among them J1 HRO_TYPE-C-31-M-12, J2 Conn_ARM_JTAG_SWD_10, J3 JST_S2B-PH-SM4-TB, Q1 AO3407, SW1 JS202011JCQN, SW2 KSC721J, SW3 RotaryEncoder_Switch, U1 USBLC6-2SC6, U2 MAX17263xxTE, U3 MCP73831-2-OT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

Commit message: Fix resistor numbering
Parts:
- renumbered R7 to R6, R8 to R7
Changed lines of the file:
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@@
   (symbol (lib_id "Device:R_Small") (at 173.99 109.22 270) (mirror x) (unit 1)
     (in_bom yes) (on_board yes)
-    (property "Reference" "R8" (id 0) (at 173.99 104.242 90))
+    (property "Reference" "R7" (id 0) (at 173.99 104.242 90))
     (property "Value" "100" (id 1) (at 173.99 106.553 90))
     (property "Footprint" "Resistor_SMD:R_0603_1608Metric_Pad0.98x0.95mm_HandSolder" (id 2) (at 173.99 109.22 0)
@@
   (symbol (lib_id "Device:R_Small") (at 245.11 138.43 0) (mirror y) (unit 1)
     (in_bom yes) (on_board yes)
-    (property "Reference" "R7" (id 0) (at 246.609 137.262 0)
+    (property "Reference" "R6" (id 0) (at 246.609 137.262 0)
       (effects (font (size 1.27 1.27)) (justify right))
     )
@@
     )
     (path "/00000000-0000-0000-0000-00005faf9a8f"
-      (reference "R7") (unit 1) (value "3.9k") (footprint "Resistor_SMD:R_0603_1608Metric_Pad0.98x0.95mm_HandSolder")
+      (reference "R6") (unit 1) (value "3.9k") (footprint "Resistor_SMD:R_0603_1608Metric_Pad0.98x0.95mm_HandSolder")
     )
     (path "/00000000-0000-0000-0000-00005fb532b0"
-      (reference "R8") (unit 1) (value "100") (footprint "Resistor_SMD:R_0603_1608Metric_Pad0.98x0.95mm_HandSolder")
+      (reference "R7") (unit 1) (value "100") (footprint "Resistor_SMD:R_0603_1608Metric_Pad0.98x0.95mm_HandSolder")
     )
     (path "/00000000-0000-0000-0000-00005f8da76e"

Commit message: Add title block to schematic
Other:
- title: (none) -> NumBLE Wireless Numpad
Changed lines of the file:
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@@
 (kicad_sch (version 20210406) (generator eeschema)
   (paper "A4")
+  (title_block
+    (title "NumBLE Wireless Numpad")
+    (date "2021-05-31")
+    (rev "1.0")
+  )
   (junction (at 38.1 50.8) (diameter 1.016) (color 0 0 0 0))
   (junction (at 39.37 172.72) (diameter 1.016) (color 0 0 0 0))
